File: GT232_CYPRESS_TQFP/GT232_CYPRESS_TQFP.kicad_sch (KiCad schematic)
At the start: 33 parts, among them IC1 CY8C4014LQI-421, IC2 CY8C4014LQI-422, IC3 CY8C4024LQI-S401, J1 Conn_01x05, U1 LMR51610XDBVR

Commit message: Aggiornato schema e PCB del modello con micro 4014
Parts:
- removed IC1: CY8C4014LQI-421, QFN50P300X300X60-17N-D, symbol CY8C4014SXA:CY8C4014LQI-421
- removed R2: 10K, Resistor_SMD:R_0603_1608Metric_Pad0.98x0.95mm_HandSolder, symbol Device:R
- added J2: Conn_01x05, Connector_PinHeader_2.54mm:PinHeader_1x05_P2.54mm_Vertical, symbol Connector_Generic:Conn_01x05
Connections:
- net 12V: now also J1.1 (Pin_1); no longer J1.4 (Pin_4)
- net 5V: now also C7.1, C8.1, C9.1, IC2.6 (VCCD), IC2.7 (VDD), J2.2 (Pin_2)
- net GND: now also C14.2, C9.2, IC2.25 (EP), J1.3 (Pin_3), J2.4 (Pin_4); no longer J1.5 (Pin_5)
- net SW_C: now also IC2.22 (P3.1/SWD_CL), J2.3 (Pin_3); no longer J1.3 (Pin_3)
- net SW_D: now also IC2.21 (P3.0/SWD_IO), J2.1 (Pin_1); no longer J1.2 (Pin_2)
- net TX: no longer J1.1 (Pin_1)
- net XRES: now also C14.1, IC2.24 (XRES), J2.5 (Pin_5); no longer C14.2
- no-connect marks 27 -> 16
Other:
- moved on the sheet: C14, C9, IC3, R13, R35, R36
