File: GT232_CY8C4124LQI-443/GT232_CY8C4124LQI-443.kicad_pcb (KiCad board)
At the start: 4 copper layers, 50.7 x 13.8 mm, 31 parts, among them IC2 CY8C4124LQI-443, J1 Conn_01x05, J2 Conn_01x05, Q1 BCR573, Q2 DTC113ZCA, Q3 DTC113ZCA, Q4 DTC113ZCA, U1 LMR51610XDBVR

Commit message: update
Routing:
- net Net-(D2-K2): track 14.8 -> 13.9 mm
- net 12V: track 24.3 -> 25.0 mm
Changed lines of the file:
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@@
 	)
 	(segment
-		(start 125.552852 99.7883)
-		(end 124.7838 99.7883)
+		(start 127.763326 100.735826)
+		(end 127.763326 101.998774)
 		(width 0.254)
 		(layer "B.Cu")
@@
 	)
 	(segment
-		(start 127.6563 105.685852)
-		(end 128.8478 104.494352)
+		(start 124.7838 99.7883)
+		(end 126.8158 99.7883)
 		(width 0.254)
 		(layer "B.Cu")
@@
 	)
 	(segment
-		(start 128.8478 104.494352)
+		(start 127.6563 106.8218)
+		(end 127.6563 108.3633)
+		(width 0.254)
+		(layer "B.Cu")
+		(net "12V")
+	)
+	(segment
+		(start 127.763326 101.998774)
 		(end 128.8478 103.083248)
 		(width 0.254)
@@
 	(segment
 		(start 128.8478 103.083248)
-		(end 125.552852 99.7883)
+		(end 128.8478 105.6303)
 		(width 0.254)
 		(layer "B.Cu")
@@
 	)
 	(segment
-		(start 127.6563 108.3633)
-		(end 127.6563 105.685852)
+		(start 126.8158 99.7883)
+		(end 127.763326 100.735826)
+		(width 0.254)
+		(layer "B.Cu")
+		(net "12V")
+	)
+	(segment
+		(start 128.8478 105.6303)
+		(end 127.6563 106.8218)
 		(width 0.254)
 		(layer "B.Cu")
@@
 	)
 	(segment
-		(start 129.416339 101.685182)
-		(end 129.416339 107.468839)
-		(width 0.254)
-		(layer "B.Cu")
-		(net "Net-(D2-K2)")
-	)
-	(segment
 		(start 134.9438 107.2813)
 		(end 136.7218 107.2813)
@@
 	)
 	(segment
+		(start 134.5628 107.6623)
+		(end 134.9438 107.2813)
+		(width 0.254)
+		(layer "B.Cu")
+		(net "Net-(D2-K2)")
+	)
+	(segment
 		(start 136.7218 107.2813)
 		(end 137.4838 108.0433)
@@
 	)
 	(segment
+		(start 131.2608 107.6623)
+		(end 134.5628 107.6623)
+		(width 0.254)
+		(layer "B.Cu")
+		(net "Net-(D2-K2)")
+	)
+	(segment
 		(start 137.4838 108.0433)
 		(end 137.4838 108.4883)
@@
 	)
 	(segment
-		(start 129.416339 107.468839)
-		(end 129.6098 107.6623)
+		(start 129.416339 101.685182)
+		(end 129.416339 105.817839)
 		(width 0.254)
 		(layer "B.Cu")
@@
 	)
 	(segment
-		(start 134.5628 107.6623)
-		(end 134.9438 107.2813)
-		(width 0.254)
-		(layer "B.Cu")
-		(net "Net-(D2-K2)")
-	)
-	(segment
-		(start 129.6098 107.6623)
-		(end 134.5628 107.6623)
+		(start 129.416339 105.817839)
+		(end 131.2608 107.6623)
 		(width 0.254)
 		(layer "B.Cu")
@@
 	)
 	(segment
+		(start 128.3398 103.2173)
+		(end 127.4508 102.3283)
+		(width 0.254)
+		(layer "B.Cu")
+		(net "PNP")
+	)
+	(segment
+		(start 127.4508 102.3283)
+		(end 124.7838 102.3283)
+		(width 0.254)
+		(layer "B.Cu")
+		(net "PNP")
+	)
+	(segment
+		(start 126.3078 107.2813)
+		(end 128.3398 105.2493)
+		(width 0.254)
+		(layer "B.Cu")
+		(net "PNP")
+	)
+	(segment
+		(start 129.5313 109.3133)
+		(end 126.8158 109.3133)
+		(width 0.254)
+		(layer "B.Cu")
+		(net "PNP")
+	)
+	(segment
+		(start 126.8158 109.3133)
+		(end 126.3078 108.8053)
+		(width 0.254)
+		(layer "B.Cu")
+		(net "PNP")
+	)
+	(segment
 		(start 126.3078 108.8053)
 		(end 126.3078 107.2813)
@@
 	)
 	(segment
-		(start 126.3078 107.2813)
-		(end 127.1968 106.3923)
-		(width 0.254)
-		(layer "B.Cu")
-		(net "PNP")
-	)
-	(segment
-		(start 127.4508 102.3283)
-		(end 124.7838 102.3283)
-		(width 0.254)
-		(layer "B.Cu")
-		(net "PNP")
-	)
-	(segment
-		(start 128.3398 104.3603)
+		(start 128.3398 105.2493)
 		(end 128.3398 103.2173)
 		(width 0.254)
 		(layer "B.Cu")
-		(net "PNP")
-	)
-	(segment
-		(start 127.1968 105.5033)
-		(end 128.3398 104.3603)
-		(width 0.254)
-		(layer "B.Cu")
-		(net "PNP")
-	)
-	(segment
-		(start 127.1968 106.3923)
-		(end 127.1968 105.5033)
-		(width 0.254)
-		(layer "B.Cu")
-		(net "PNP")
-	)
-	(segment
-		(start 126.8158 109.3133)
-		(end 126.3078 108.8053)
-		(width 0.254)
-		(layer "B.Cu")
-		(net "PNP")
-	)
-	(segment
-		(start 129.5313 109.3133)
-		(end 126.8158 109.3133)
-		(width 0.254)
-		(layer "B.Cu")
-		(net "PNP")
-	)
-	(segment
-		(start 128.3398 103.2173)
-		(end 127.4508 102.3283)
-		(width 0.254)
-		(layer "B.Cu")
